File: schematic/diy_arduino_esp01/diy_arduino_esp01.kicad_sch (KiCad schematic)
At the start: 28 parts, among them J10 3.3v, J11 gnd, J2 CP0102, J3 Barrel_Jack, J4 D5, J5 RFID, J7 Anaolg Pins, J8 RFID, J9 5V, SW1 SW_Push, SW2 hardware interupt, U1 ATmega328-P, U2 LM7805_TO220, U3 ESP-01, U4 LM1117T-3.3, Y1 Crystal

Commit message: final schematic
Parts:
- removed C5, C6: 16V 10uF, Capacitor_THT:CP_Radial_D5.0mm_P2.00mm, symbol Device:C_Polarized
- removed U4: LM1117T-3.3, Package_TO_SOT_THT:TO-220F-3_Vertical, symbol Regulator_Linear:LM1117T-3.3
- added J1: 3.3v, Connector_PinSocket_2.54mm:PinSocket_1x03_P2.54mm_Vertical, symbol Connector:Conn_01x03_Socket
Connections:
- net 3.3V: now also J1.2 (Pin_2)
- net 5V: now also J1.1 (Pin_1)
- net GND: now also J1.3 (Pin_3)
